File: kicad/serv_vpr_template.kicad_pcb (KiCad board)
At the start: 2 copper layers, 0 parts

Commit message: add (very rough) keepout to template
Other:
- board text added: "0"
- board text added: "7"
Changed lines of the file:
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@@
     (effects (font (size 15 15) (thickness 3) bold) (justify left bottom))
   )
+  (gr_text "7" (at 76.65 -180.9) (layer "User.9")
+    (effects (font (size 100 100) (thickness 20) bold) (justify left bottom))
+  )
+  (gr_text "0" (at 173.4 -181.05) (layer "User.9")
+    (effects (font (size 100 100) (thickness 20) bold) (justify left bottom))
+  )
+  (zone (net 0) (net_name "") (layers "F&B.Cu") (name "7") (hatch edge 0.5)
+    (connect_pads (clearance 0))
+    (min_thickness 0.25) (filled_areas_thickness no)
+    (keepout (tracks not_allowed) (vias not_allowed) (pads not_allowed) (copperpour not_allowed) (footprints allowed))
+    (fill (thermal_gap 0.5) (thermal_bridge_width 0.5))
+    (polygon
+      (pts
+        (xy 99.45 -304.65)
+        (xy 168.45 -304.65)
+        (xy 174.15 -302.85)
+        (xy 177.3 -298.8)
+        (xy 177.9 -293.4)
+        (xy 176.25 -288.45)
+        (xy 133.05 -188.55)
+        (xy 129.9 -185.55)
+        (xy 127.05 -184.35)
+        (xy 123.3 -184.05)
+        (xy 119.4 -185.7)
+        (xy 116.4 -188.1)
+        (xy 114.75 -192)
+        (xy 114.45 -196.05)
+        (xy 152.55 -284.25)
+        (xy 99.75 -284.25)
+        (xy 96.3 -285.3)
+        (xy 92.25 -288.75)
+        (xy 90.75 -293.4)
+        (xy 90.9 -296.1)
+        (xy 93.15 -300.45)
+        (xy 96.3 -303.15)
+        (xy 98.7 -304.5)
+      )
+    )
+  )
+  (zone (net 0) (net_name "") (layers "F&B.Cu") (name "0") (hatch edge 0.5)
+    (connect_pads (clearance 0))
+    (min_thickness 0.25) (filled_areas_thickness no)
+    (keepout (tracks not_allowed) (vias not_allowed) (pads not_allowed) (copperpour not_allowed) (footprints not_allowed))
+    (fill (thermal_gap 0.5) (thermal_bridge_width 0.5))
+    (polygon
+      (pts
+        (xy 192.75 -258.6)
+        (xy 197.85 -280.5)
+        (xy 204.15 -291.15)
+        (xy 210.3 -297.9)
+        (xy 224.1 -304.95)
+        (xy 237 -304.65)
+        (xy 252.45 -297.15)
+        (xy 265.8 -278.1)
+        (xy 269.7 -255.9)
+        (xy 269.7 -232.65)
+        (xy 264.75 -210.75)
+        (xy 257.85 -198)
+        (xy 251.85 -190.95)
+        (xy 237.75 -184.05)
+        (xy 223.8 -184.5)
+        (xy 209.7 -191.55)
+        (xy 197.55 -209.7)
+        (xy 192.6 -231.9)
+      )
+    )
+  )
 )

Commit message: add more IO things to template
Parts:
- added C500: 100n, Capacitor_THT:C_Disc_D5.1mm_W3.2mm_P5.00mm, F.Cu at (31.5, 3.00)
- added D1: ~, LED_THT:LED_D5.0mm, F.Cu at (24.0, -447.0)
- added D10: ~, LED_THT:LED_D5.0mm, F.Cu at (53.0, -439.0)
- added D11: ~, LED_THT:LED_D5.0mm, F.Cu at (60.5, -447.0)
- added D12: ~, LED_THT:LED_D5.0mm, F.Cu at (60.5, -439.0)
- added D13: ~, LED_THT:LED_D5.0mm, F.Cu at (68.0, -447.0)
- added D14: ~, LED_THT:LED_D5.0mm, F.Cu at (68.0, -439.0)
- added D15: ~, LED_THT:LED_D5.0mm, F.Cu at (75.5, -447.0)
- added D16: ~, LED_THT:LED_D5.0mm, F.Cu at (75.5, -439.0)
- added D17: ~, LED_THT:LED_D5.0mm, F.Cu at (84.0, -447.0)
- added D18: ~, LED_THT:LED_D5.0mm, F.Cu at (84.0, -439.0)
- added D19: ~, LED_THT:LED_D5.0mm, F.Cu at (91.5, -447.0)
- added D2: ~, LED_THT:LED_D5.0mm, F.Cu at (24.0, -439.0)
- added D20: ~, LED_THT:LED_D5.0mm, F.Cu at (91.5, -439.0)
- added D21: ~, LED_THT:LED_D5.0mm, F.Cu at (99.0, -447.0)
- added D22: ~, LED_THT:LED_D5.0mm, F.Cu at (99.0, -439.0)
- added D23: ~, LED_THT:LED_D5.0mm, F.Cu at (106.5, -447.0)
- added D24: ~, LED_THT:LED_D5.0mm, F.Cu at (106.5, -439.0)
- added D25: ~, LED_THT:LED_D5.0mm, F.Cu at (115.0, -447.0)
- added D26: ~, LED_THT:LED_D5.0mm, F.Cu at (115.0, -439.0)
- added D27: ~, LED_THT:LED_D5.0mm, F.Cu at (122.5, -447.0)
- added D28: ~, LED_THT:LED_D5.0mm, F.Cu at (122.5, -439.0)
- added D29: ~, LED_THT:LED_D5.0mm, F.Cu at (130.0, -447.0)
- added D3: ~, LED_THT:LED_D5.0mm, F.Cu at (31.0, -447.0)
- added D30: ~, LED_THT:LED_D5.0mm, F.Cu at (130.0, -439.0)
- added D31: ~, LED_THT:LED_D5.0mm, F.Cu at (137.5, -447.0)
- added D32: ~, LED_THT:LED_D5.0mm, F.Cu at (137.5, -439.0)
- added D33: ~, LED_THT:LED_D5.0mm, F.Cu at (148.0, -447.0)
- added D34: ~, LED_THT:LED_D5.0mm, F.Cu at (148.0, -439.0)
- added D35: ~, LED_THT:LED_D5.0mm, F.Cu at (162.0, -447.0)
- added D36: ~, LED_THT:LED_D5.0mm, F.Cu at (-14.0, -0.50)
- added D37: ~, LED_THT:LED_D5.0mm, F.Cu at (158.5, -439.0)
- added D38: ~, LED_THT:LED_D5.0mm, F.Cu at (166.0, -439.0)
- added D39: ~, LED_THT:LED_D5.0mm, F.Cu at (173.5, -439.0)
- added D4: ~, LED_THT:LED_D5.0mm, F.Cu at (31.0, -439.0)
- added D40: ~, LED_THT:LED_D5.0mm, F.Cu at (181.0, -439.0)
- added D41: ~, LED_THT:LED_D5.0mm, F.Cu at (191.5, -447.0)
- added D42: ~, LED_THT:LED_D5.0mm, F.Cu at (195.0, -439.0)
- added D43: ~, LED_THT:LED_D5.0mm, F.Cu at (199.0, -447.0)
- added D44: ~, LED_THT:LED_D5.0mm, F.Cu at (202.5, -439.0)
- added D45: ~, LED_THT:LED_D5.0mm, F.Cu at (206.5, -447.0)
- added D46: ~, LED_THT:LED_D5.0mm, F.Cu at (210.0, -439.0)
- added D47: ~, LED_THT:LED_D5.0mm, F.Cu at (214.0, -447.0)
- added D48: ~, LED_THT:LED_D5.0mm, F.Cu at (217.5, -439.0)
- added D5: ~, LED_THT:LED_D5.0mm, F.Cu at (38.0, -447.0)
- added D6: ~, LED_THT:LED_D5.0mm, F.Cu at (38.0, -439.0)
- added D7: ~, LED_THT:LED_D5.0mm, F.Cu at (45.0, -447.0)
- added D8: ~, LED_THT:LED_D5.0mm, F.Cu at (45.0, -439.0)
- added D9: ~, LED_THT:LED_D5.0mm, F.Cu at (53.0, -447.0)
- added J1: Conn_01x02_Pin, Connector_Wago:Wago_734-132_1x02_P3.50mm_Vertical, F.Cu at (12.0, -447.0)
- added R1: 10k, Resistor_THT:R_Axial_DIN0207_L6.3mm_D2.5mm_P10.16mm_Horizontal, F.Cu at (27.0, 17.1)
- added R2: 10k, Resistor_THT:R_Axial_DIN0207_L6.3mm_D2.5mm_P10.16mm_Horizontal, F.Cu at (47.0, 17.1)
- added R3: 10k, Resistor_THT:R_Axial_DIN0207_L6.3mm_D2.5mm_P10.16mm_Horizontal, F.Cu at (67.0, 17.1)
- added R4: 10k, Resistor_THT:R_Axial_DIN0207_L6.3mm_D2.5mm_P10.16mm_Horizontal, F.Cu at (189.0, 17.0)
- added R5: 10k, Resistor_THT:R_Axial_DIN0207_L6.3mm_D2.5mm_P10.16mm_Horizontal, F.Cu at (309.0, 17.0)
- added R6: 10k, Resistor_THT:R_Axial_DIN0207_L6.3mm_D2.5mm_P10.16mm_Horizontal, F.Cu at (31.0, 17.1)
- added RN1: SIL 9-8 10K, Resistor_THT:R_Array_SIP9, F.Cu at (77.2, 4.00)
- added RN10: SIL 8-4 1,0K, Resistor_THT:R_Array_SIP8, F.Cu at (37.0, -452.5)
- added RN11: SIL 8-4 1,0K, Resistor_THT:R_Array_SIP8, F.Cu at (52.0, -452.5)
- added RN12: SIL 8-4 1,0K, Resistor_THT:R_Array_SIP8, F.Cu at (67.0, -452.5)
- added RN13: SIL 8-4 1,0K, Resistor_THT:R_Array_SIP8, F.Cu at (83.0, -452.5)
- added RN14: SIL 8-4 1,0K, Resistor_THT:R_Array_SIP8, F.Cu at (98.0, -452.5)
- added RN15: SIL 8-4 1,0K, Resistor_THT:R_Array_SIP8, F.Cu at (114.0, -452.5)
- added RN16: SIL 8-4 1,0K, Resistor_THT:R_Array_SIP8, F.Cu at (129.0, -452.5)
- added RN17: SIL 8-4 1,0K, Resistor_THT:R_Array_SIP8, F.Cu at (147.0, -452.5)
- added RN18: SIL 8-4 1,0K, Resistor_THT:R_Array_SIP8, F.Cu at (161.0, -452.5)
- added RN19: SIL 8-4 1,0K, Resistor_THT:R_Array_SIP8, F.Cu at (190.5, -452.5)
- added RN2: SIL 9-8 10K, Resistor_THT:R_Array_SIP9, F.Cu at (102.1, 4.00)
- added RN20: SIL 8-4 1,0K, Resistor_THT:R_Array_SIP8, F.Cu at (205.5, -452.5)
- added RN3: SIL 9-8 10K, Resistor_THT:R_Array_SIP9, F.Cu at (127.1, 4.00)
- added RN4: SIL 9-8 10K, Resistor_THT:R_Array_SIP9, F.Cu at (152.0, 4.00)
- added RN5: SIL 9-8 10K, Resistor_THT:R_Array_SIP9, F.Cu at (197.2, 4.00)
- added RN6: SIL 9-8 10K, Resistor_THT:R_Array_SIP9, F.Cu at (222.1, 4.00)
- added RN7: SIL 9-8 10K, Resistor_THT:R_Array_SIP9, F.Cu at (247.1, 4.00)
- added RN8: SIL 9-8 10K, Resistor_THT:R_Array_SIP9, F.Cu at (272.0, 4.00)
- added RN9: SIL 8-4 1,0K, Resistor_THT:R_Array_SIP8, F.Cu at (23.0, -452.5)
- added SW1: ~, Button_Switch_THT:SW_PUSH_6mm_H5mm, F.Cu at (15.8, 9.75)
- added SW10: ~, Button_Switch_THT:SW_DIP_SPSTx08_Slide_9.78x22.5mm_W7.62mm_P2.54mm, F.Cu at (249.0, 16.0)
- added SW11: ~, Button_Switch_THT:SW_DIP_SPSTx08_Slide_9.78x22.5mm_W7.62mm_P2.54mm, F.Cu at (273.9, 16.0)
- added SW12: ~, Button_Switch_THT:SW_PUSH_6mm_H5mm, F.Cu at (177.5, 9.67)
- added SW13: ~, Button_Switch_THT:SW_PUSH_6mm_H5mm, F.Cu at (297.5, 9.67)
- added SW2: ~, Button_Switch_THT:SW_PUSH_6mm_H5mm, F.Cu at (35.8, 9.75)
- added SW3: ~, Button_Switch_THT:SW_PUSH_6mm_H5mm, F.Cu at (55.8, 9.75)
- added SW4: ~, Button_Switch_THT:SW_DIP_SPSTx08_Slide_9.78x22.5mm_W7.62mm_P2.54mm, F.Cu at (79.1, 16.0)
- added SW5: ~, Button_Switch_THT:SW_DIP_SPSTx08_Slide_9.78x22.5mm_W7.62mm_P2.54mm, F.Cu at (104.0, 16.0)
- added SW6: ~, Button_Switch_THT:SW_DIP_SPSTx08_Slide_9.78x22.5mm_W7.62mm_P2.54mm, F.Cu at (129.0, 16.0)
- added SW7: ~, Button_Switch_THT:SW_DIP_SPSTx08_Slide_9.78x22.5mm_W7.62mm_P2.54mm, F.Cu at (153.9, 16.0)
- added SW8: ~, Button_Switch_THT:SW_DIP_SPSTx08_Slide_9.78x22.5mm_W7.62mm_P2.54mm, F.Cu at (199.1, 16.0)
- added SW9: ~, Button_Switch_THT:SW_DIP_SPSTx08_Slide_9.78x22.5mm_W7.62mm_P2.54mm, F.Cu at (224.0, 16.0)

Commit message: add remaining IOs to template
Parts:
- removed D36: ~, LED_THT:LED_D5.0mm
- added D49: ~, LED_THT:LED_D5.0mm, F.Cu at (237.9, -447.0)
- added D50: ~, LED_THT:LED_D5.0mm, F.Cu at (241.4, -439.0)
- added D51: ~, LED_THT:LED_D5.0mm, F.Cu at (245.4, -447.0)
- added D52: ~, LED_THT:LED_D5.0mm, F.Cu at (248.9, -439.0)
- added D53: ~, LED_THT:LED_D5.0mm, F.Cu at (252.9, -447.0)
- added D54: ~, LED_THT:LED_D5.0mm, F.Cu at (256.4, -439.0)
- added D55: ~, LED_THT:LED_D5.0mm, F.Cu at (260.4, -447.0)
- added D56: ~, LED_THT:LED_D5.0mm, F.Cu at (263.9, -439.0)
- added D57: ~, LED_THT:LED_D5.0mm, F.Cu at (269.8, -447.0)
- added D58: ~, LED_THT:LED_D5.0mm, F.Cu at (273.3, -439.0)
- added D59: ~, LED_THT:LED_D5.0mm, F.Cu at (277.3, -447.0)
- added D60: ~, LED_THT:LED_D5.0mm, F.Cu at (280.8, -439.0)
- added D61: ~, LED_THT:LED_D5.0mm, F.Cu at (284.8, -447.0)
- added D62: ~, LED_THT:LED_D5.0mm, F.Cu at (288.3, -439.0)
- added D63: ~, LED_THT:LED_D5.0mm, F.Cu at (292.3, -447.0)
- added D64: ~, LED_THT:LED_D5.0mm, F.Cu at (295.8, -439.0)
- added D65: ~, LED_THT:LED_D5.0mm, F.Cu at (302.5, -447.0)
- added D66: ~, LED_THT:LED_D5.0mm, F.Cu at (306.0, -439.0)
- added D67: ~, LED_THT:LED_D5.0mm, F.Cu at (310.0, -447.0)
- added D68: ~, LED_THT:LED_D5.0mm, F.Cu at (313.5, -439.0)
- added D69: ~, LED_THT:LED_D5.0mm, F.Cu at (317.5, -447.0)
- added D70: ~, LED_THT:LED_D5.0mm, F.Cu at (321.0, -439.0)
- added D71: ~, LED_THT:LED_D5.0mm, F.Cu at (325.0, -447.0)
- added D72: ~, LED_THT:LED_D5.0mm, F.Cu at (328.5, -439.0)
- added RN21: SIL 8-4 1,0K, Resistor_THT:R_Array_SIP8, F.Cu at (236.9, -452.5)
- added RN22: SIL 8-4 1,0K, Resistor_THT:R_Array_SIP8, F.Cu at (251.9, -452.5)
- added RN23: SIL 8-4 1,0K, Resistor_THT:R_Array_SIP8, F.Cu at (268.8, -452.5)
- added RN24: SIL 8-4 1,0K, Resistor_THT:R_Array_SIP8, F.Cu at (283.8, -452.5)
- added RN25: SIL 8-4 1,0K, Resistor_THT:R_Array_SIP8, F.Cu at (301.5, -452.5)
- added RN26: SIL 8-4 1,0K, Resistor_THT:R_Array_SIP8, F.Cu at (316.5, -452.5)
- moved D25 14.2 mm to (129.2, -447.0)
- moved D26 14.2 mm to (129.2, -439.0)
- moved D27 14.2 mm to (136.7, -447.0)
- moved D28 14.2 mm to (136.7, -439.0)
- moved D29 14.2 mm to (144.2, -447.0)
- moved D30 14.2 mm to (144.2, -439.0)
- moved D31 14.2 mm to (151.7, -447.0)
- moved D32 14.2 mm to (151.7, -439.0)
- moved D33 14.2 mm to (162.2, -447.0)
- moved D34 14.2 mm to (162.2, -439.0)
- moved D37 14.2 mm to (172.7, -439.0)
- moved D38 14.2 mm to (180.2, -439.0)
- moved D39 14.2 mm to (187.7, -439.0)
- moved D40 14.2 mm to (195.2, -439.0)
- moved D41 14.2 mm to (205.7, -447.0)
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Connections:
- net Net-(RN4-R7) renamed /i_ibus_rdt_1
- D37 pad 2: /o_dbus_sel_0 -> /o_dbus_sel_3
- D38 pad 2: /o_dbus_sel_1 -> /o_dbus_sel_2
- D39 pad 2: /o_dbus_sel_2 -> /o_dbus_sel_1
- D40 pad 2: /o_dbus_sel_3 -> /o_dbus_sel_0
- RN1 pad 2: /i_ibus_rdt_0 -> /i_ibus_rdt_31
- RN4 pad 9: Net-(RN4-R8) -> /i_ibus_rdt_0
- SW1 pad 2: Net-(R1-Pad2) -> GND
- SW12 pad 2: /i_dbus_ack -> VCC
- SW13 pad 2: /d_dbus_ack -> VCC
- SW2 pad 2: /i_rst -> VCC
- SW3 pad 2: /i_timer_irq -> VCC
- SW4 pad 16: /i_ibus_rdt_0 -> /i_ibus_rdt_31
- SW7 pad 9: Net-(RN4-R8) -> /i_ibus_rdt_0
Other:
- board text added: "+5V"
- board text added: "1"
- board text added: "10"
- board text added: "11"
- board text added: "12"
- board text added: "13"
- board text added: "14"
- board text added: "15"
- board text added: "16"
- board text added: "17"
- board text added: "18"
- board text added: "19"
- board text added: "2"
- board text added: "20"
- board text added: "21"
- board text added: "22"
- board text added: "23"
- board text added: "24"
- board text added: "25"
- board text added: "26"
- board text added: "27"
- board text added: "28"
- board text added: "29"
- board text added: "3"
- board text added: "30"
- board text added: "31"
- board text added: "4"
- board text added: "5"
- board text added: "6"
- board text added: "8"
- board text added: "9"
- board text added: "ACTIVE"
- board text added: "DBUS ADDR"
- board text added: "DBUS read data"
- board text added: "DBUS write"
- board text added: "DBUS write data"
- board text added: "GND"
- board text added: "IBUS ADDR"
- board text added: "IBUS read data"
- board text added: "WR_BYTE_ENA[3:0]"
- board text added: "WR_ENA"
- board text added: "acknowledge"
- board text added: "clock"
- board text added: "reset"
- board text added: "timer irq"

Commit message: move upper part of template up by one row
Parts:
- moved D1 25.0 mm to (34.4, -472.0)
- moved D10 25.0 mm to (64.7, -464.0)
- moved D11 25.0 mm to (72.2, -472.0)
- moved D12 25.0 mm to (72.2, -464.0)
- moved D13 25.0 mm to (79.7, -472.0)
- moved D14 25.0 mm to (79.7, -464.0)
- moved D15 25.0 mm to (87.2, -472.0)
- moved D16 25.0 mm to (87.2, -464.0)
- moved D17 25.0 mm to (96.9, -472.0)
- moved D18 25.0 mm to (96.9, -464.0)
- moved D19 25.0 mm to (104.4, -472.0)
- moved D2 25.0 mm to (34.4, -464.0)
- moved D20 25.0 mm to (104.4, -464.0)
- moved D21 25.0 mm to (111.9, -472.0)
- moved D22 25.0 mm to (111.9, -464.0)
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
Commit message: connect ibus/dbus read data in template
Connections:
- net Net-(RN1-R2) renamed /i_ibus_rdt_30
- net Net-(RN1-R3) renamed /i_ibus_rdt_29
- net Net-(RN1-R4) renamed /i_ibus_rdt_28
- net Net-(RN1-R5) renamed /i_ibus_rdt_27
- net Net-(RN1-R6) renamed /i_ibus_rdt_26
- net Net-(RN1-R7) renamed /i_ibus_rdt_25
- net Net-(RN1-R8) renamed /i_ibus_rdt_24
- net Net-(RN2-R1) renamed /i_ibus_rdt_23
- net Net-(RN2-R2) renamed /i_ibus_rdt_22
- net Net-(RN2-R3) renamed /i_ibus_rdt_21
- net Net-(RN2-R4) renamed /i_ibus_rdt_20
- net Net-(RN2-R5) renamed /i_ibus_rdt_19
- net Net-(RN2-R6) renamed /i_ibus_rdt_18
- net Net-(RN2-R7) renamed /i_ibus_rdt_17
- net Net-(RN2-R8) renamed /i_ibus_rdt_16
- net Net-(RN3-R1) renamed /i_ibus_rdt_15
- net Net-(RN3-R2) renamed /i_ibus_rdt_14
- net Net-(RN3-R3) renamed /i_ibus_rdt_13
- net Net-(RN3-R4) renamed /i_ibus_rdt_12
- net Net-(RN3-R5) renamed /i_ibus_rdt_11
- net Net-(RN3-R6) renamed /i_ibus_rdt_10
- net Net-(RN3-R7) renamed /i_ibus_rdt_9
- net Net-(RN3-R8) renamed /i_ibus_rdt_8
- net Net-(RN4-R1) renamed /i_ibus_rdt_7
- net Net-(RN4-R2) renamed /i_ibus_rdt_6
- net Net-(RN4-R3) renamed /i_ibus_rdt_5
- net Net-(RN4-R4) renamed /i_ibus_rdt_4
- net Net-(RN4-R5) renamed /i_ibus_rdt_3
- net Net-(RN4-R6) renamed /i_ibus_rdt_2
- net Net-(RN5-R2) renamed /i_dbus_rdt_30
- net Net-(RN5-R3) renamed /i_dbus_rdt_29
- net Net-(RN5-R4) renamed /i_dbus_rdt_28
- net Net-(RN5-R5) renamed /i_dbus_rdt_27
- net Net-(RN5-R6) renamed /i_dbus_rdt_26
- net Net-(RN5-R7) renamed /i_dbus_rdt_25
- net Net-(RN5-R8) renamed /i_dbus_rdt_24
- net Net-(RN6-R1) renamed /i_dbus_rdt_23
- net Net-(RN6-R2) renamed /i_dbus_rdt_22
- net Net-(RN6-R3) renamed /i_dbus_rdt_21
- net Net-(RN6-R4) renamed /i_dbus_rdt_20
- net Net-(RN6-R5) renamed /i_dbus_rdt_19
- net Net-(RN6-R6) renamed /i_dbus_rdt_18
- net Net-(RN6-R7) renamed /i_dbus_rdt_17
- net Net-(RN6-R8) renamed /i_dbus_rdt_16
- net Net-(RN7-R1) renamed /i_dbus_rdt_15
- net Net-(RN7-R2) renamed /i_dbus_rdt_14
- net Net-(RN7-R3) renamed /i_dbus_rdt_13
- net Net-(RN7-R4) renamed /i_dbus_rdt_12
- net Net-(RN7-R5) renamed /i_dbus_rdt_11
- net Net-(RN7-R6) renamed /i_dbus_rdt_10
- net Net-(RN7-R7) renamed /i_dbus_rdt_9
- net Net-(RN7-R8) renamed /i_dbus_rdt_8
- net Net-(RN8-R1) renamed /i_dbus_rdt_7
- net Net-(RN8-R2) renamed /i_dbus_rdt_6
- net Net-(RN8-R3) renamed /i_dbus_rdt_5
- net Net-(RN8-R4) renamed /i_dbus_rdt_4
- net Net-(RN8-R5) renamed /i_dbus_rdt_3
- net Net-(RN8-R6) renamed /i_dbus_rdt_2
- net Net-(RN8-R7) renamed /i_dbus_rdt_1
- RN5 pad 2: /i_dbus_rdt_0 -> /i_dbus_rdt_31
- RN8 pad 9: Net-(RN8-R8) -> /i_dbus_rdt_0
- SW11 pad 9: Net-(RN8-R8) -> /i_dbus_rdt_0
- SW8 pad 16: /i_dbus_rdt_0 -> /i_dbus_rdt_31
